File: kicad/toprebox_prototype.kicad_pcb (KiCad board)
At the start: 2 copper layers, 282.1 x 103.7 mm, 42 parts

Commit message: completed matrix
Parts:
- added C5: 100n, Capacitor_SMD:C_0402_1005Metric, F.Cu at (559.4, 1.83)
- added C6: 100n, Capacitor_SMD:C_0402_1005Metric, F.Cu at (559.4, 3.80)
- added C7: 220p, Capacitor_SMD:C_0402_1005Metric, F.Cu at (559.4, 5.77)
- added C8: 100n, Capacitor_SMD:C_0402_1005Metric, F.Cu at (559.4, 7.74)
- added JP2: Ext_Res, Resistor_SMD:R_0603_1608Metric_Pad0.98x0.95mm_HandSolder, F.Cu at (555.9, 17.6)
- added R18: 100k, Resistor_SMD:R_0402_1005Metric, F.Cu at (546.4, 10.8)
- added R19: 100k, Resistor_SMD:R_0402_1005Metric, F.Cu at (546.4, 12.8)
- added R20: 100k, Resistor_SMD:R_0402_1005Metric, F.Cu at (546.4, 14.8)
- added R21: 100k, Resistor_SMD:R_0402_1005Metric, F.Cu at (546.4, 16.8)
- added R22: 100k, Resistor_SMD:R_0402_1005Metric, F.Cu at (546.4, 18.8)
- added R23: 100k, Resistor_SMD:R_0402_1005Metric, F.Cu at (546.4, 20.8)
- added R24: 100k, Resistor_SMD:R_0402_1005Metric, F.Cu at (549.3, 10.8)
- added R25: 100k, Resistor_SMD:R_0402_1005Metric, F.Cu at (549.3, 12.8)
- added R26: 100k, Resistor_SMD:R_0402_1005Metric, F.Cu at (549.3, 14.8)
- added R27: 100k, Resistor_SMD:R_0402_1005Metric, F.Cu at (549.3, 16.8)
- added R28: 100k, Resistor_SMD:R_0402_1005Metric, F.Cu at (549.3, 18.8)
- added R29: 100k, Resistor_SMD:R_0402_1005Metric, F.Cu at (549.3, 20.8)
- added R30: 100k, Resistor_SMD:R_0402_1005Metric, F.Cu at (552.2, 10.8)
- added R31: 100k, Resistor_SMD:R_0402_1005Metric, F.Cu at (552.2, 12.8)
- added R32: 100k, Resistor_SMD:R_0402_1005Metric, F.Cu at (552.2, 14.8)
- added R33: 1k, Resistor_SMD:R_0402_1005Metric, F.Cu at (552.2, 16.8)
- added R34: 100k, Resistor_SMD:R_0402_1005Metric, F.Cu at (552.2, 18.8)
- added SW_EC1: Topre, footprints:Topre, F.Cu at (445.5, -53.2)
- added SW_EC10: Topre, footprints:Topre, F.Cu at (460.5, -8.21)
- added SW_EC11: Topre, footprints:Topre, F.Cu at (460.5, 6.79)
- added SW_EC12: Topre, footprints:Topre, F.Cu at (460.5, 21.8)
- added SW_EC13: Topre, footprints:Topre, F.Cu at (475.5, -53.2)
- added SW_EC14: Topre, footprints:Topre, F.Cu at (475.5, -38.2)
- added SW_EC15: Topre, footprints:Topre, F.Cu at (475.5, -23.2)
- added SW_EC16: Topre, footprints:Topre, F.Cu at (475.5, -8.21)
- added SW_EC17: Topre, footprints:Topre, F.Cu at (475.5, 6.79)
- added SW_EC18: Topre, footprints:Topre, F.Cu at (475.5, 21.8)
- added SW_EC19: Topre, footprints:Topre, F.Cu at (490.5, -53.2)
- added SW_EC2: Topre, footprints:Topre, F.Cu at (445.5, -38.2)
- added SW_EC20: Topre, footprints:Topre, F.Cu at (490.5, -38.2)
- added SW_EC21: Topre, footprints:Topre, F.Cu at (490.5, -23.2)
- added SW_EC22: Topre, footprints:Topre, F.Cu at (490.5, -8.21)
- added SW_EC23: Topre, footprints:Topre, F.Cu at (490.5, 6.79)
- added SW_EC24: Topre, footprints:Topre, F.Cu at (490.5, 21.8)
- added SW_EC25: Topre, footprints:Topre, F.Cu at (505.5, -53.2)
- added SW_EC26: Topre, footprints:Topre, F.Cu at (505.5, -38.2)
- added SW_EC27: Topre, footprints:Topre, F.Cu at (505.5, -23.2)
- added SW_EC28: Topre, footprints:Topre, F.Cu at (505.5, -8.21)
- added SW_EC29: Topre, footprints:Topre, F.Cu at (505.5, 6.79)
- added SW_EC3: Topre, footprints:Topre, F.Cu at (445.5, -23.2)
- added SW_EC30: Topre, footprints:Topre, F.Cu at (505.5, 21.8)
- added SW_EC31: Topre, footprints:Topre, F.Cu at (520.5, -53.2)
- added SW_EC32: Topre, footprints:Topre, F.Cu at (520.5, -38.2)
- added SW_EC33: Topre, footprints:Topre, F.Cu at (520.5, -23.2)
- added SW_EC34: Topre, footprints:Topre, F.Cu at (520.5, -8.21)
- added SW_EC35: Topre, footprints:Topre, F.Cu at (520.5, 6.79)
- added SW_EC36: Topre, footprints:Topre, F.Cu at (520.5, 21.8)
- added SW_EC37: Topre, footprints:Topre, F.Cu at (535.5, -53.2)
- added SW_EC38: Topre, footprints:Topre, F.Cu at (535.5, -38.2)
- added SW_EC39: Topre, footprints:Topre, F.Cu at (535.5, -23.2)
- added SW_EC4: Topre, footprints:Topre, F.Cu at (445.5, -8.21)
- added SW_EC40: Topre, footprints:Topre, F.Cu at (535.5, -8.21)
- added SW_EC41: Topre, footprints:Topre, F.Cu at (535.5, 6.79)
- added SW_EC42: Topre, footprints:Topre, F.Cu at (535.5, 21.8)
- added SW_EC5: Topre, footprints:Topre, F.Cu at (445.5, 6.79)
- added SW_EC6: Topre, footprints:Topre, F.Cu at (445.5, 21.8)
- added SW_EC7: Topre, footprints:Topre, F.Cu at (460.5, -53.2)
- added SW_EC8: Topre, footprints:Topre, F.Cu at (460.5, -38.2)
- added SW_EC9: Topre, footprints:Topre, F.Cu at (460.5, -23.2)
- added U1: YAAJ_BlackPill_Part_Like, footprints:YAAJ_BlackPill_1, F.Cu at (549.0, -51.8)
- added U5: 74HC4051, footprints:TSSOP16, F.Cu at (548.2, 5.21)
- added U6: 74HC4051, footprints:TSSOP16, F.Cu at (554.7, 5.21)
- added U7: OPA350, Package_SO:SOIC-8_3.9x4.9mm_P1.27mm, F.Cu at (557.9, 13.2)
- renumbered S1 to SW_EC1, S2 to SW_EC2, S3 to SW_EC3, S6 to SW_EC4, S5 to SW_EC5, S4 to SW_EC6, S9 to SW_EC7, S8 to SW_EC8

Commit message: replaced half of the matrix
Parts:
- removed S22, S23, S24, S25, S26, S27, S28, S29, S30, S31, S32, S33, S34, S35, S36, S37, S38, S39, S40, S41, S42: , footprints:Topre
- removed the SW_EC1 at (445.5, -53.2)
- removed the SW_EC2 at (445.5, -38.2)
- removed the SW_EC3 at (9.84, -36.7)
- removed the SW_EC3 at (445.5, -23.2)
- removed the SW_EC4 at (445.5, -8.21)
- removed the SW_EC4 at (28.2, -31.8)
- removed the SW_EC5 at (445.5, 6.79)
- removed the SW_EC5 at (23.3, -13.4)
- removed the SW_EC6 at (18.4, 4.92)
- removed the SW_EC6 at (445.5, 21.8)
- removed the SW_EC7 at (54.1, -36.0)
- removed the SW_EC7 at (460.5, -53.2)
- removed the SW_EC8 at (47.6, -18.1)
- removed the SW_EC8 at (460.5, -38.2)
- removed U1: YAAJ_BlackPill_Part_Like, footprints:YAAJ_BlackPill_1
- added S1: , footprints:Topre, B.Cu at (268.5, 0.00)
- added S2: , footprints:Topre, B.Cu at (263.6, -18.4)
- added S3: , footprints:Topre, B.Cu at (258.7, -36.7)
- added S4: , footprints:Topre, B.Cu at (250.2, 4.92)
- added S5: , footprints:Topre, B.Cu at (245.3, -13.4)
- added S6: , footprints:Topre, B.Cu at (240.4, -31.8)
- added S8: , footprints:Topre, B.Cu at (219.8, -17.5)
- added S9: , footprints:Topre, B.Cu at (212.7, -35.1)
- added SW_EC3: Topre, footprints:Topre, B.Cu at (9.84, -36.7)
- added SW_EC4: Topre, footprints:Topre, B.Cu at (28.2, -31.8)
- added SW_EC5: Topre, footprints:Topre, B.Cu at (23.3, -13.4)
- added SW_EC6: Topre, footprints:Topre, B.Cu at (18.4, 4.92)
- added SW_EC7: Topre, footprints:Topre, B.Cu at (55.9, -35.1)
- added SW_EC8: Topre, footprints:Topre, B.Cu at (48.7, -17.5)
- added U2: BlackPill_STLINK, footprints:WeAct_BlackPill_without_SWD_First_Row, B.Cu at (141.7, -50.7)
- C5, C6, C7, C8, JP2, R18, R19, R20, R21, R22, R23, R24, R25, R26, R27, R28, R29, R30, R31, R32, R33, R34, S10, S11, S12, S13, S14, S15, S16, S17, S18, S19, S20, S21, S7, SW_EC10, SW_EC11, SW_EC12, SW_EC13, SW_EC14, SW_EC15, SW_EC16, SW_EC17, SW_EC18, SW_EC19, SW_EC20, SW_EC21, SW_EC22, SW_EC23, SW_EC24, SW_EC25, SW_EC26, SW_EC27, SW_EC28, SW_EC29, SW_EC30, SW_EC31, SW_EC32, SW_EC33, SW_EC34, SW_EC35, SW_EC36, SW_EC37, SW_EC38, SW_EC39, SW_EC40, SW_EC41, SW_EC42, SW_EC9, U5, U6, U7: moved to B.Cu
- SW_EC1, SW_EC2: value (none) -> Topre; moved to B.Cu
- moved SW_EC19 448.2 mm to (49.1, 24.7), turned to 152.5 degrees
- moved C5 435.4 mm to (124.0, 5.26), turned to 180 degrees
- moved C6 435.4 mm to (124.0, 7.23), turned to 180 degrees
- moved C7 435.4 mm to (124.0, 9.20), turned to 180 degrees
- moved C8 435.4 mm to (124.0, 11.2), turned to 180 degrees
- moved U7 432.4 mm to (125.5, 16.6), turned to 180 degrees
- moved JP2 428.3 mm to (127.6, 21.1), turned to 180 degrees
- moved SW_EC20 428.3 mm to (68.5, 34.8), turned to 152.5 degrees
- moved U6 426.0 mm to (128.7, 8.64), turned to 180 degrees
- moved R30 421.0 mm to (131.2, 14.2), turned to 180 degrees
- moved R31 421.0 mm to (131.2, 16.2), turned to 180 degrees
- moved R32 421.0 mm to (131.2, 18.2), turned to 180 degrees
- moved R33 421.0 mm to (131.2, 20.2), turned to 180 degrees
- moved R34 421.0 mm to (131.2, 22.2), turned to 180 degrees
- moved SW_EC9 419.5 mm to (41.6, 0.14), turned to 158 degrees
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Connections:
- SW_EC1 pad 1: (no net) -> Net-(SW_EC1-Pad1)
- SW_EC1 pad 2: outerpinky_bottom -> Net-(SW_EC1-Pad2)
- SW_EC1 pad 3: (no net) -> GND
- SW_EC2 pad 1: (no net) -> Net-(SW_EC11-Pad1)
- SW_EC2 pad 2: outerpinky_home -> Net-(SW_EC1-Pad2)
- SW_EC2 pad 3: (no net) -> GND
Other:
- board size 282.1 x 103.7 mm -> 301.6 x 116 mm

Commit message: matrix complete
Parts:
- removed S1, S10, S11, S12, S13, S14, S15, S16, S17, S18, S19, S2, S20, S21, S3, S4, S5, S6, S7, S8, S9: , footprints:Topre
- added R1: 100k, Resistor_SMD:R_0402_1005Metric, F.Cu at (127.1, 6.58)
- C5, C6, C7, C8, JP2, R18, R19, R20, R21, R22, R23, R24, R25, R26, R27, R28, R29, R30, R31, R32, R33, R34, U5, U7: moved to F.Cu
- moved SW_EC40 137.8 mm to (180.7, 44.9), turned to -152.5 degrees
- moved SW_EC39 126.7 mm to (268.5, 0.00), turned to -165 degrees
- moved SW_EC38 123.7 mm to (263.6, -18.4), turned to -165 degrees
- moved SW_EC41 118.7 mm to (200.1, 34.8), turned to -152.5 degrees
- moved SW_EC36 89.8 mm to (250.2, 4.92), turned to -165 degrees
- moved SW_EC42 78.7 mm to (219.5, 24.7), turned to -152.5 degrees
- moved SW_EC24 59.1 mm to (176.1, 25.8), turned to -152.5 degrees
- moved SW_EC33 58.5 mm to (226.9, 0.14), turned to -158 degrees
- moved SW_EC30 56.0 mm to (207.4, 2.62), turned to -158 degrees
- moved SW_EC27 55.7 mm to (192.1, 15.3), turned to -152.5 degrees
- moved SW_EC23 54.4 mm to (167.4, 8.99), turned to -152.5 degrees
- moved SW_EC32 54.2 mm to (219.8, -17.5), turned to -158 degrees
- moved SW_EC29 51.7 mm to (200.3, -15.0), turned to -158 degrees
- moved SW_EC26 51.4 mm to (183.3, -1.55), turned to -152.5 degrees
- moved SW_EC22 50.9 mm to (158.6, -7.86), turned to -152.5 degrees
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- renumbered SW_EC3 to SW_EC1, SW_EC1 to SW_EC3, SW_EC35 to SW_EC34, SW_EC36 to SW_EC35, SW_EC37 to SW_EC36, SW_EC39 to SW_EC37, SW_EC40 to SW_EC38, SW_EC41 to SW_EC39, SW_EC34 to SW_EC40, SW_EC38 to SW_EC41
Connections:
- net Net-(SW_EC1-Pad1) renamed R2
- net Net-(SW_EC10-Pad1) renamed R0
- net Net-(SW_EC11-Pad1) renamed R1
- net Net-(SW_EC19-Pad1) renamed R3
- net Net-(SW_EC28-Pad2) renamed C8
- net Net-(SW_EC31-Pad2) renamed C9
- net Net-(SW_EC35-Pad2) renamed C10
- net Net-(SW_EC39-Pad2) renamed C11
- R18 pad 1: Net-(U5-A0) -> C0
- R19 pad 1: Net-(U5-A1) -> C1
- R20 pad 1: Net-(U5-A2) -> C2
- R21 pad 1: Net-(U5-A3) -> C3
- R23 pad 1: Net-(U5-A4) -> C4
- R25 pad 1: Net-(U5-A5) -> C5
- R31 pad 1: Net-(U6-A6) -> C7
- SW_EC1 pad 2: Net-(SW_EC1-Pad2) -> C0
- SW_EC10 pad 2: Net-(SW_EC10-Pad2) -> C3
- SW_EC11 pad 2: Net-(SW_EC10-Pad2) -> C3
- SW_EC12 pad 2: Net-(SW_EC10-Pad2) -> C3
- SW_EC13 pad 2: Net-(SW_EC13-Pad2) -> C4
- SW_EC14 pad 2: Net-(SW_EC13-Pad2) -> C4
- SW_EC15 pad 2: Net-(SW_EC13-Pad2) -> C4
- SW_EC16 pad 2: Net-(SW_EC16-Pad2) -> C5
- SW_EC17 pad 2: Net-(SW_EC16-Pad2) -> C5
- SW_EC18 pad 2: Net-(SW_EC16-Pad2) -> C5
- SW_EC19 pad 2: Net-(SW_EC10-Pad2) -> C3
- SW_EC2 pad 2: Net-(SW_EC1-Pad2) -> C0
- SW_EC20 pad 2: Net-(SW_EC13-Pad2) -> C4
- SW_EC21 pad 2: Net-(SW_EC16-Pad2) -> C5
- SW_EC22 pad 2: Net-(SW_EC22-Pad2) -> C6
- SW_EC23 pad 2: Net-(SW_EC22-Pad2) -> C6
- SW_EC24 pad 2: Net-(SW_EC22-Pad2) -> C6
- SW_EC25 pad 2: Net-(SW_EC25-Pad2) -> C7
- SW_EC26 pad 2: Net-(SW_EC25-Pad2) -> C7
- SW_EC27 pad 2: Net-(SW_EC25-Pad2) -> C7
- SW_EC3 pad 2: Net-(SW_EC1-Pad2) -> C0
- SW_EC4 pad 2: Net-(SW_EC4-Pad2) -> C1
- SW_EC40 pad 2: Net-(SW_EC22-Pad2) -> C6
- SW_EC41 pad 2: Net-(SW_EC25-Pad2) -> C7
- SW_EC5 pad 2: Net-(SW_EC4-Pad2) -> C1
- SW_EC6 pad 2: Net-(SW_EC4-Pad2) -> C1
- SW_EC7 pad 2: Net-(SW_EC7-Pad2) -> C2
- SW_EC8 pad 2: Net-(SW_EC7-Pad2) -> C2
- SW_EC9 pad 2: Net-(SW_EC7-Pad2) -> C2
- U5 pad 1: Net-(U5-A4) -> C4
- U5 pad 12: Net-(U5-A3) -> C3
- U5 pad 13: Net-(U5-A0) -> C0
- U5 pad 14: Net-(U5-A1) -> C1
- U5 pad 15: Net-(U5-A2) -> C2
- U5 pad 5: Net-(U5-A5) -> C5
- U6 pad 1: GND -> C6
- U6 pad 2: Net-(U6-A6) -> C7

Commit message: stuff
Parts:
- removed R1, R18: 100k, Resistor_SMD:R_0402_1005Metric
- added H1: MountingHole, footprints:HOLE_M2, F.Cu at (-2.68, -40.5)
- added H10: MountingHole, footprints:HOLE_M2, F.Cu at (73.5, 48.8)
- added H11: MountingHole, footprints:HOLE_M2, F.Cu at (122.1, 7.74)
- added H12: MountingHole, footprints:HOLE_M2, F.Cu at (122.1, 10.9)
- added H13: MountingHole, footprints:HOLE_M2, F.Cu at (122.1, 14.1)
- added H14: MountingHole, footprints:HOLE_M2, F.Cu at (122.1, 17.3)
- added H15: MountingHole, footprints:HOLE_M2, F.Cu at (122.1, 20.5)
- added H16: MountingHole, footprints:HOLE_M2, F.Cu at (125.3, 7.74)
- added H17: MountingHole, footprints:HOLE_M2, F.Cu at (125.3, 10.9)
- added H18: MountingHole, footprints:HOLE_M2, F.Cu at (125.3, 14.1)
- added H19: MountingHole, footprints:HOLE_M2, F.Cu at (125.3, 17.3)
- added H2: MountingHole, footprints:HOLE_M2, F.Cu at (40.8, -30.4)
- added H2: MountingHole, footprints:HOLE_M2_funny, F.Cu at (180.7, -33.0)
- added H3: MountingHole, footprints:HOLE_M2, F.Cu at (88.4, -33.0)
- added H4: MountingHole, footprints:HOLE_M2, F.Cu at (115.2, 5.95)
- added H5: MountingHole, footprints:HOLE_M2, F.Cu at (56.3, -9.52)
- added H6: MountingHole, footprints:HOLE_M2, F.Cu at (6.55, 12.8)
- added H7: MountingHole, footprints:HOLE_M2, F.Cu at (33.9, 14.9)
- added H8: MountingHole, footprints:HOLE_M2, F.Cu at (63.1, 20.2)
- added H9: MountingHole, footprints:HOLE_M2, F.Cu at (98.8, 38.1)
- added R35: 100k, Resistor_SMD:R_0402_1005Metric, B.Cu at (102.4, -82.2)
- added R36: 100k, Resistor_SMD:R_0402_1005Metric, B.Cu at (102.4, -80.2)
- C5, C8, JP2, R19, R20, R21, R22, R23, R24, R25, R26, R27, R29, R30, R31, R32, R34: moved to B.Cu
- C6: value 100n -> 220p; moved to B.Cu
- C7: value 220p -> 100n; moved to B.Cu
- R28: value 100k -> 1k; moved to B.Cu
- R33: value 1k -> 100k; moved to B.Cu
- U2: value BlackPill_STLINK -> 74HC4051; footprint footprints:WeAct_BlackPill_without_SWD_First_Row -> footprints:TSSOP16
- U5: value 74HC4051 -> Helios; footprint footprints:TSSOP16 -> footprints:RP2040_Pro_Micro
- U6: value 74HC4051 -> OPA350; footprint footprints:TSSOP16 -> Package_SO:SOIC-8_3.9x4.9mm_P1.27mm
- U7: value OPA350 -> 74HC4051; footprint Package_SO:SOIC-8_3.9x4.9mm_P1.27mm -> footprints:TSSOP16; moved to B.Cu
- moved R33 101.4 mm to (102.4, -86.2), turned to 180 degrees
- moved R34 101.4 mm to (102.4, -84.2), turned to 180 degrees
- moved U6 100.1 mm to (105.4, -60.9), turned to 180 degrees
- moved R26 99.8 mm to (105.3, -86.2), turned to 180 degrees
- moved R28 99.8 mm to (105.3, -82.2), turned to 180 degrees
- moved R29 99.8 mm to (105.3, -80.2), turned to 180 degrees
- moved R27 99.8 mm to (105.3, -84.2), turned to 180 degrees
- moved R30 99.8 mm to (105.3, -78.2), turned to 180 degrees
- moved R19 98.5 mm to (108.2, -86.2), turned to 180 degrees
- moved R21 98.5 mm to (108.2, -82.2), turned to 180 degrees
- moved R22 98.5 mm to (108.2, -80.2), turned to 180 degrees
- moved R20 98.5 mm to (108.2, -84.2), turned to 180 degrees
- moved R23 98.5 mm to (108.2, -78.2), turned to 180 degrees
- moved U7 95.0 mm to (99.9, -68.9), turned to 180 degrees
- moved R31 87.3 mm to (105.3, -76.2), turned to 180 degrees
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Connections:
- C6 pad 1: GND -> APLEX_OUT_PIN_0
- C6 pad 2: +3V3 -> GND
- C7 pad 1: APLEX_OUT_PIN_0 -> GND
- C7 pad 2: GND -> +3V3
- R19 pad 1: C1 -> ADC
- R19 pad 2: GND -> Net-(JP2-B)
- R20 pad 1: C2 -> C0
- R21 pad 1: C3 -> C1
- R22 pad 1: Net-(U6-A0) -> C2
- R23 pad 1: C4 -> C3
- R24 pad 1: Net-(U6-A1) -> C4
- R26 pad 1: Net-(U6-A2) -> Net-(U2-A6)
- R27 pad 1: Net-(U5-A6) -> Net-(U2-A7)
- R28 pad 1: Net-(U6-A3) -> Net-(JP2-B)
- R29 pad 1: Net-(U5-A7) -> Net-(U7-A0)
- R30 pad 1: Net-(U6-A5) -> Net-(U7-A1)
- R31 pad 1: C7 -> Net-(U7-A2)
- R32 pad 1: Net-(U6-A7) -> Net-(U7-A3)
- R33 pad 1: Net-(JP2-B) -> C6
- R34 pad 1: ADC -> Net-(U7-A5)
- R34 pad 2: Net-(JP2-B) -> GND
- U2 pad 10: unconnected-(U2-PA15-Pad10) -> AMUX_SEL_1
- U2 pad 11: unconnected-(U2-PB3-Pad11) -> AMUX_SEL_0
- U2 pad 12: unconnected-(U2-PB4-Pad12) -> C3
- U2 pad 13: unconnected-(U2-PB5-Pad13) -> C0
- U2 pad 14: unconnected-(U2-PB6-Pad14) -> C1
- U2 pad 15: unconnected-(U2-PB7-Pad15) -> C2
- U2 pad 16: unconnected-(U2-PB8-Pad16) -> +3V3
- U2 pad 2: unconnected-(U2-PB13-Pad2) -> Net-(U2-A6)
- U2 pad 3: unconnected-(U2-PB14-Pad3) -> APLEX_OUT_PIN_0
- U2 pad 4: unconnected-(U2-PB15-Pad4) -> Net-(U2-A7)
- U2 pad 5: unconnected-(U2-PA8-Pad5) -> C5
- U2 pad 6: unconnected-(U2-PA9-Pad6) -> APLEX_EN_PIN_0
- U2 pad 7: unconnected-(U2-PA10-Pad7) -> GND
- U2 pad 8: unconnected-(U2-PA11-Pad8) -> GND
- U2 pad 9: unconnected-(U2-PA12-Pad9) -> AMUX_SEL_2
- U5 pad 1: C4 -> unconnected-(U5-P0-Pad1)
- U5 pad 10: AMUX_SEL_1 -> unconnected-(U5-P7-Pad10)
- U5 pad 11: AMUX_SEL_0 -> unconnected-(U5-P8-Pad11)
- U5 pad 12: C3 -> unconnected-(U5-P9-Pad12)
- U5 pad 13: C0 -> unconnected-(U5-5V-Pad13)
- U5 pad 14: C1 -> GND
- U5 pad 15: C2 -> unconnected-(U5-RST-Pad15)
- U5 pad 2: Net-(U5-A6) -> unconnected-(U5-P1-Pad2)
- U5 pad 3: APLEX_OUT_PIN_0 -> GND
- U5 pad 4: Net-(U5-A7) -> GND
- U5 pad 5: C5 -> unconnected-(U5-P2-Pad5)
- U5 pad 6: APLEX_EN_PIN_0 -> unconnected-(U5-P3-Pad6)
- U5 pad 7: GND -> unconnected-(U5-P4-Pad7)
- U5 pad 8: GND -> unconnected-(U5-P5-Pad8)
- U5 pad 9: AMUX_SEL_2 -> unconnected-(U5-P6-Pad9)
- U6 pad 1: C6 -> (no net)
- U6 pad 2: C7 -> Net-(JP2-B)
- U6 pad 4: Net-(U6-A7) -> GND
- U6 pad 5: Net-(U6-A5) -> (no net)
- U6 pad 6: APLEX_EN_PIN_1 -> ADC
- U6 pad 7: GND -> +3V3
- U6 pad 8: GND -> (no net)
- U7 pad 1: (no net) -> C6
- U7 pad 2: Net-(JP2-B) -> C7
- U7 pad 4: GND -> Net-(U7-A7)
- U7 pad 5: (no net) -> Net-(U7-A5)
- U7 pad 6: ADC -> APLEX_EN_PIN_1
- U7 pad 7: +3V3 -> GND
- U7 pad 8: (no net) -> GND

Commit message: new plate outline
Parts:
- removed C5, C7, C8: 100n, Capacitor_SMD:C_0402_1005Metric
- removed C6: 220p, Capacitor_SMD:C_0402_1005Metric
- removed H1, H10, H11, H12, H13, H14, H15, H16, H17, H18, H19, H2, H3, H4, H5, H6, H7, H8, H9: MountingHole, footprints:HOLE_M2
- removed H2: MountingHole, footprints:HOLE_M2_funny
- removed JP2: Ext_Res, Resistor_SMD:R_0603_1608Metric_Pad0.98x0.95mm_HandSolder
- removed R19, R20, R21, R22, R23, R24, R25, R26, R27, R29, R30, R31, R32, R33, R34, R35, R36: 100k, Resistor_SMD:R_0402_1005Metric
- removed R28: 1k, Resistor_SMD:R_0402_1005Metric
- removed SW_EC1, SW_EC10, SW_EC11, SW_EC12, SW_EC13, SW_EC14, SW_EC15, SW_EC16, SW_EC17, SW_EC18, SW_EC19, SW_EC2, SW_EC20, SW_EC21, SW_EC22, SW_EC23, SW_EC24, SW_EC25, SW_EC26, SW_EC27, SW_EC28, SW_EC29, SW_EC3, SW_EC30, SW_EC31, SW_EC32, SW_EC33, SW_EC34, SW_EC35, SW_EC36, SW_EC37, SW_EC38, SW_EC39, SW_EC4, SW_EC40, SW_EC41, SW_EC42, SW_EC5, SW_EC6, SW_EC7, SW_EC8, SW_EC9: Topre, footprints:Topre
- removed U2, U7: 74HC4051, footprints:TSSOP16
- removed U5: Helios, footprints:RP2040_Pro_Micro
- removed U6: OPA350, Package_SO:SOIC-8_3.9x4.9mm_P1.27mm
- added S1: , MX, F.Cu at (0.00, 0.00)
- added S10: , MX, F.Cu at (60.5, 4.18)
- added S11: , MX, F.Cu at (67.8, -13.4)
- added S12: , MX, F.Cu at (75.1, -30.9)
- added S13: , MX, F.Cu at (75.8, 17.0)
- added S14: , MX, F.Cu at (85.1, 0.46)
- added S15: , MX, F.Cu at (94.5, -16.1)
- added S16: , MX, F.Cu at (88.9, 32.4)
- added S17: , MX, F.Cu at (98.2, 15.9)
- added S18: , MX, F.Cu at (107.6, -0.63)
- added S19: , MX, F.Cu at (45.6, 29.8)
- added S2: , MX, F.Cu at (5.71, -18.1)
- added S20: , MX, F.Cu at (64.6, 40.6)
- added S21: , MX, F.Cu at (83.6, 51.3)
- added S22: , MX, F.Cu at (12.4, -55.9)
- added S23: , MX, F.Cu at (30.5, -50.2)
- added S24: , MX, F.Cu at (53.5, -56.5)
- added S25: , MX, F.Cu at (73.0, -54.5)
- added S26: , MX, F.Cu at (91.7, -44.3)
- added S27: , MX, F.Cu at (106.7, -31.6)
- added S28: , MX, F.Cu at (277.4, 0.00)
- added S29: , MX, F.Cu at (271.7, -18.1)
- added S3: , MX, F.Cu at (11.4, -36.2)
- added S30: , MX, F.Cu at (266.0, -36.2)
- added S31: , MX, F.Cu at (259.3, 5.71)
- added S32: , MX, F.Cu at (253.6, -12.4)
- added S33: , MX, F.Cu at (247.9, -30.5)
- added S34: , MX, F.Cu at (236.4, 1.53)
- added S35: , MX, F.Cu at (229.1, -16.0)
- added S36: , MX, F.Cu at (221.8, -33.6)
- added S37: , MX, F.Cu at (216.9, 4.18)
- added S38: , MX, F.Cu at (209.6, -13.4)
- added S39: , MX, F.Cu at (202.4, -30.9)
- added S4: , MX, F.Cu at (18.1, 5.71)
- added S40: , MX, F.Cu at (201.7, 17.0)
- added S41: , MX, F.Cu at (192.3, 0.46)
- added S42: , MX, F.Cu at (182.9, -16.1)
- added S43: , MX, F.Cu at (188.6, 32.4)
- added S44: , MX, F.Cu at (179.2, 15.9)
- added S45: , MX, F.Cu at (169.9, -0.63)
- added S46: , MX, F.Cu at (231.8, 29.8)
- added S47: , MX, F.Cu at (212.8, 40.6)
- added S48: , MX, F.Cu at (193.8, 51.3)
- added S49: , MX, F.Cu at (265.1, -55.9)
- added S5: , MX, F.Cu at (23.8, -12.4)
- added S50: , MX, F.Cu at (246.9, -50.2)
- added S51: , MX, F.Cu at (224.0, -56.5)
- added S52: , MX, F.Cu at (204.4, -54.5)
- added S53: , MX, F.Cu at (185.7, -44.3)
- added S54: , MX, F.Cu at (170.8, -31.6)
- added S6: , MX, F.Cu at (29.5, -30.5)
- added S7: , MX, F.Cu at (41.0, 1.53)
- added S8: , MX, F.Cu at (48.3, -16.0)
- added S9: , MX, F.Cu at (55.6, -33.6)
Other:
- board size 301.6 x 116 mm -> 325.1 x 138.2 mm
- net class Default added: clearance 0.2, trace_width 0.25, via_dia 0.8, via_drill 0.4
