File: kicad/toprebox_prototype.kicad_pcb (KiCad board)
At the start: 2 copper layers, 325.1 x 138.2 mm, 54 parts

Commit message: re did the pcb
Parts:
- removed S1, S10, S11, S12, S13, S14, S15, S16, S17, S18, S19, S2, S20, S21, S22, S23, S24, S25, S26, S27, S3, S4, S5, S6, S7, S8, S9: , MX
- added C5: 100n, Capacitor_SMD:C_0402_1005Metric, B.Cu at (227.0, 77.8)
- added C6: 220p, Capacitor_SMD:C_0402_1005Metric, B.Cu at (227.0, 79.8)
- added C7: 100n, Capacitor_SMD:C_0402_1005Metric, B.Cu at (227.0, 81.8)
- added C8: 100n, Capacitor_SMD:C_0402_1005Metric, B.Cu at (227.0, 83.7)
- added H1: MountingHole, footprints:HOLE_M2, B.Cu at (254.5, 114.7)
- added H10: MountingHole, footprints:HOLE_M2, B.Cu at (251.3, 127.5)
- added H11: MountingHole, footprints:HOLE_M2, B.Cu at (248.1, 114.7)
- added H12: MountingHole, footprints:HOLE_M2, B.Cu at (248.1, 117.9)
- added H13: MountingHole, footprints:HOLE_M2, B.Cu at (248.1, 121.1)
- added H14: MountingHole, footprints:HOLE_M2, B.Cu at (248.1, 124.3)
- added H15: MountingHole, footprints:HOLE_M2, B.Cu at (248.1, 127.5)
- added H16: MountingHole, footprints:HOLE_M2, B.Cu at (244.9, 114.7)
- added H17: MountingHole, footprints:HOLE_M2, B.Cu at (244.9, 117.9)
- added H18: MountingHole, footprints:HOLE_M2, B.Cu at (244.9, 121.1)
- added H19: MountingHole, footprints:HOLE_M2, B.Cu at (244.9, 124.3)
- added H2: MountingHole, footprints:HOLE_M2, B.Cu at (254.5, 117.9)
- added H3: MountingHole, footprints:HOLE_M2, B.Cu at (254.5, 121.1)
- added H4: MountingHole, footprints:HOLE_M2, B.Cu at (254.5, 124.3)
- added H5: MountingHole, footprints:HOLE_M2, B.Cu at (254.5, 127.5)
- added H6: MountingHole, footprints:HOLE_M2, B.Cu at (251.3, 114.7)
- added H7: MountingHole, footprints:HOLE_M2, B.Cu at (251.3, 117.9)
- added H8: MountingHole, footprints:HOLE_M2, B.Cu at (251.3, 121.1)
- added H9: MountingHole, footprints:HOLE_M2, B.Cu at (251.3, 124.3)
- added JP2: Ext_Res, Resistor_SMD:R_0603_1608Metric_Pad0.98x0.95mm_HandSolder, B.Cu at (235.0, 107.6)
- added R19: 100k, Resistor_SMD:R_0402_1005Metric, B.Cu at (235.7, 77.8)
- added R20: 100k, Resistor_SMD:R_0402_1005Metric, B.Cu at (235.7, 79.8)
- added R21: 100k, Resistor_SMD:R_0402_1005Metric, B.Cu at (235.7, 81.8)
- added R22: 100k, Resistor_SMD:R_0402_1005Metric, B.Cu at (235.7, 83.8)
- added R23: 100k, Resistor_SMD:R_0402_1005Metric, B.Cu at (235.7, 85.8)
- added R24: 100k, Resistor_SMD:R_0402_1005Metric, B.Cu at (235.7, 87.8)
- added R25: 100k, Resistor_SMD:R_0402_1005Metric, B.Cu at (235.7, 89.8)
- added R26: 100k, Resistor_SMD:R_0402_1005Metric, B.Cu at (232.8, 77.8)
- added R27: 100k, Resistor_SMD:R_0402_1005Metric, B.Cu at (232.8, 79.8)
- added R28: 1k, Resistor_SMD:R_0402_1005Metric, B.Cu at (232.8, 81.8)
- added R29: 100k, Resistor_SMD:R_0402_1005Metric, B.Cu at (232.8, 83.8)
- added R30: 100k, Resistor_SMD:R_0402_1005Metric, B.Cu at (232.8, 85.8)
- added R31: 100k, Resistor_SMD:R_0402_1005Metric, B.Cu at (232.8, 87.8)
- added R32: 100k, Resistor_SMD:R_0402_1005Metric, B.Cu at (232.8, 89.8)
- added R33: 100k, Resistor_SMD:R_0402_1005Metric, B.Cu at (229.9, 77.8)
- added R34: 100k, Resistor_SMD:R_0402_1005Metric, B.Cu at (229.9, 79.8)
- added R35: 100k, Resistor_SMD:R_0402_1005Metric, B.Cu at (229.9, 81.8)
- added R36: 100k, Resistor_SMD:R_0402_1005Metric, B.Cu at (229.9, 83.8)
- added SW_EC1: Topre, footprints:Topre, B.Cu at (12.4, -55.9)
- added SW_EC10: Topre, footprints:Topre, B.Cu at (55.6, -33.6)
- added SW_EC11: Topre, footprints:Topre, B.Cu at (48.3, -16.0)
- added SW_EC12: Topre, footprints:Topre, B.Cu at (41.0, 1.53)
- added SW_EC13: Topre, footprints:Topre, B.Cu at (73.0, -54.5)
- added SW_EC14: Topre, footprints:Topre, B.Cu at (75.1, -30.9)
- added SW_EC15: Topre, footprints:Topre, B.Cu at (67.8, -13.4)
- added SW_EC16: Topre, footprints:Topre, B.Cu at (60.5, 4.18)
- added SW_EC17: Topre, footprints:Topre, B.Cu at (45.6, 29.8)
- added SW_EC18: Topre, footprints:Topre, B.Cu at (91.7, -44.3)
- added SW_EC19: Topre, footprints:Topre, B.Cu at (94.5, -16.1)
- added SW_EC2: Topre, footprints:Topre, B.Cu at (11.4, -36.2)
- added SW_EC20: Topre, footprints:Topre, B.Cu at (85.1, 0.46)
- added SW_EC21: Topre, footprints:Topre, B.Cu at (75.8, 17.0)
- added SW_EC22: Topre, footprints:Topre, B.Cu at (64.6, 40.6)
- added SW_EC23: Topre, footprints:Topre, B.Cu at (106.7, -31.6)
- added SW_EC24: Topre, footprints:Topre, B.Cu at (107.6, -0.63)
- added SW_EC25: Topre, footprints:Topre, B.Cu at (98.2, 15.9)
- added SW_EC26: Topre, footprints:Topre, B.Cu at (88.9, 32.4)
- added SW_EC27: Topre, footprints:Topre, B.Cu at (83.6, 51.3)
- added SW_EC28: Topre, footprints:Topre, B.Cu at (295.6, 84.3)
- added SW_EC29: Topre, footprints:Topre, B.Cu at (295.6, 99.3)
- added SW_EC3: Topre, footprints:Topre, B.Cu at (5.71, -18.1)
- added SW_EC30: Topre, footprints:Topre, B.Cu at (295.6, 114.3)
- added SW_EC31: Topre, footprints:Topre, B.Cu at (295.6, 129.3)
- added SW_EC32: Topre, footprints:Topre, B.Cu at (295.6, 144.3)
- added SW_EC33: Topre, footprints:Topre, B.Cu at (295.6, 159.3)
- added SW_EC34: Topre, footprints:Topre, B.Cu at (295.6, 174.3)
- added SW_EC35: Topre, footprints:Topre, B.Cu at (295.6, 189.3)
- added SW_EC36: Topre, footprints:Topre, B.Cu at (295.6, 204.3)
- added SW_EC37: Topre, footprints:Topre, B.Cu at (280.6, 84.3)
- added SW_EC38: Topre, footprints:Topre, B.Cu at (280.6, 99.3)
- added SW_EC39: Topre, footprints:Topre, B.Cu at (280.6, 114.3)
- added SW_EC4: Topre, footprints:Topre, B.Cu at (0.00, 0.00)
- added SW_EC40: Topre, footprints:Topre, B.Cu at (280.6, 129.3)
- added SW_EC41: Topre, footprints:Topre, B.Cu at (280.6, 144.3)
- added SW_EC42: Topre, footprints:Topre, B.Cu at (280.6, 159.3)
- added SW_EC43: Topre, footprints:Topre, B.Cu at (280.6, 174.3)
- added SW_EC44: Topre, footprints:Topre, B.Cu at (280.6, 189.3)
- added SW_EC45: Topre, footprints:Topre, B.Cu at (280.6, 204.3)
- added SW_EC46: Topre, footprints:Topre, B.Cu at (265.6, 84.3)
- added SW_EC47: Topre, footprints:Topre, B.Cu at (265.6, 99.3)
- added SW_EC48: Topre, footprints:Topre, B.Cu at (265.6, 114.3)
- added SW_EC49: Topre, footprints:Topre, B.Cu at (265.6, 129.3)
- added SW_EC5: Topre, footprints:Topre, B.Cu at (30.5, -50.2)
- added SW_EC50: Topre, footprints:Topre, B.Cu at (265.6, 144.3)
- added SW_EC51: Topre, footprints:Topre, B.Cu at (265.6, 159.3)
- added SW_EC52: Topre, footprints:Topre, B.Cu at (265.6, 174.3)
- added SW_EC53: Topre, footprints:Topre, B.Cu at (265.6, 189.3)
- added SW_EC54: Topre, footprints:Topre, B.Cu at (265.6, 204.3)
- added SW_EC6: Topre, footprints:Topre, B.Cu at (29.5, -30.5)
- added SW_EC7: Topre, footprints:Topre, B.Cu at (23.8, -12.4)
- added SW_EC8: Topre, footprints:Topre, B.Cu at (18.1, 5.71)
- added SW_EC9: Topre, footprints:Topre, B.Cu at (53.5, -56.5)
- added U2: 74HC4051, footprints:TSSOP16, B.Cu at (233.9, 95.1)
- added U5: Helios, footprints:RP2040_Pro_Micro, B.Cu at (246.6, 95.2)
- added U6: OPA350, Package_SO:SOIC-8_3.9x4.9mm_P1.27mm, B.Cu at (232.9, 103.1)
- added U7: 74HC4051, footprints:TSSOP16, B.Cu at (227.4, 95.1)
- S28, S29, S30, S31, S32, S33, S34, S35, S36, S37, S38, S39, S40, S41, S42, S43, S44, S45, S46, S47, S48, S49, S50, S51, S52, S53, S54: footprint MX -> footprints:Topre
Other:
- net class Default removed
