File: kicad/untitled.kicad_sch (KiCad schematic)
At the start: 1 part

Commit message: completed matrix
Parts:
- added SW_EC10, SW_EC11, SW_EC12, SW_EC13, SW_EC14, SW_EC15, SW_EC16, SW_EC17, SW_EC18, SW_EC19, SW_EC2, SW_EC20, SW_EC21, SW_EC22, SW_EC23, SW_EC24, SW_EC25, SW_EC26, SW_EC27, SW_EC28, SW_EC29, SW_EC3, SW_EC30, SW_EC31, SW_EC32, SW_EC33, SW_EC34, SW_EC35, SW_EC36, SW_EC37, SW_EC38, SW_EC39, SW_EC4, SW_EC40, SW_EC41, SW_EC42, SW_EC5, SW_EC6, SW_EC7, SW_EC8, SW_EC9: Topre, footprints:Topre, symbol cipulot_parts:Topre
- SW_EC1: renamed from SW_EC2; footprint (none) -> footprints:Topre
Connections:
- net at SW_EC1.1: now also SW_EC12.1, SW_EC15.1, SW_EC18.1, SW_EC24.1, SW_EC27.1, SW_EC30.1, SW_EC33.1, SW_EC37.1, SW_EC41.1, SW_EC6.1, SW_EC9.1
- net at SW_EC1.2: now also SW_EC2.2, SW_EC3.2
- net GND: now reaches SW_EC1.3
- net GND: now also SW_EC10.3, SW_EC11.3, SW_EC12.3, SW_EC13.3, SW_EC14.3, SW_EC15.3, SW_EC16.3, SW_EC17.3, SW_EC18.3, SW_EC19.3, SW_EC2.3, SW_EC20.3, SW_EC21.3, SW_EC22.3, SW_EC23.3, SW_EC24.3, SW_EC25.3, SW_EC26.3, SW_EC27.3, SW_EC28.3, SW_EC29.3, SW_EC3.3, SW_EC30.3, SW_EC31.3, SW_EC32.3, SW_EC33.3, SW_EC34.3, SW_EC35.3, SW_EC36.3, SW_EC37.3, SW_EC38.3, SW_EC39.3, SW_EC4.3, SW_EC40.3, SW_EC41.3, SW_EC42.3, SW_EC5.3, SW_EC6.3, SW_EC7.3, SW_EC8.3, SW_EC9.3
- new net: SW_EC10.1, SW_EC13.1, SW_EC16.1, SW_EC22.1, SW_EC25.1, SW_EC28.1, SW_EC3.1, SW_EC31.1, SW_EC35.1, SW_EC39.1, SW_EC4.1, SW_EC7.1
- new net: SW_EC39.2, SW_EC40.2, SW_EC41.2
- new net: SW_EC11.1, SW_EC14.1, SW_EC17.1, SW_EC2.1, SW_EC23.1, SW_EC26.1, SW_EC29.1, SW_EC32.1, SW_EC36.1, SW_EC40.1, SW_EC5.1, SW_EC8.1
- new net: SW_EC4.2, SW_EC5.2, SW_EC6.2
- new net: SW_EC19.1, SW_EC20.1, SW_EC21.1, SW_EC34.1, SW_EC38.1, SW_EC42.1
- new net: SW_EC25.2, SW_EC26.2, SW_EC27.2, SW_EC38.2
- new net: SW_EC16.2, SW_EC17.2, SW_EC18.2, SW_EC21.2
- new net: SW_EC28.2, SW_EC29.2, SW_EC30.2, SW_EC42.2
- new net: SW_EC35.2, SW_EC36.2, SW_EC37.2
- new net: SW_EC13.2, SW_EC14.2, SW_EC15.2, SW_EC20.2
- new net: SW_EC10.2, SW_EC11.2, SW_EC12.2, SW_EC19.2
- new net: SW_EC31.2, SW_EC32.2, SW_EC33.2
- new net: SW_EC7.2, SW_EC8.2, SW_EC9.2
- new net: SW_EC22.2, SW_EC23.2, SW_EC24.2, SW_EC34.2
Other:
- moved on the sheet: SW_EC1

Commit message: matrix complete
Parts:
- renumbered SW_EC3 to SW_EC1, SW_EC1 to SW_EC3, SW_EC35 to SW_EC34, SW_EC36 to SW_EC35, SW_EC37 to SW_EC36, SW_EC39 to SW_EC37, SW_EC40 to SW_EC38, SW_EC41 to SW_EC39, SW_EC34 to SW_EC40, SW_EC38 to SW_EC41
Connections:
- net R0: now reaches SW_EC1.1, SW_EC10.1, SW_EC13.1, SW_EC16.1, SW_EC22.1, SW_EC25.1, SW_EC28.1, SW_EC31.1, SW_EC34.1, SW_EC37.1, SW_EC4.1, SW_EC7.1
- net C11: now reaches SW_EC37.2, SW_EC38.2, SW_EC39.2
- net R1: now reaches SW_EC11.1, SW_EC14.1, SW_EC17.1, SW_EC2.1, SW_EC23.1, SW_EC26.1, SW_EC29.1, SW_EC32.1, SW_EC35.1, SW_EC38.1, SW_EC5.1, SW_EC8.1
- net C1: now reaches SW_EC4.2, SW_EC5.2, SW_EC6.2
- net C0: now reaches SW_EC1.2, SW_EC2.2, SW_EC3.2
- net R3: now reaches SW_EC19.1, SW_EC20.1, SW_EC21.1, SW_EC40.1, SW_EC41.1, SW_EC42.1
- net C7: now reaches SW_EC25.2, SW_EC26.2, SW_EC27.2, SW_EC41.2
- net R2: now reaches SW_EC12.1, SW_EC15.1, SW_EC18.1, SW_EC24.1, SW_EC27.1, SW_EC3.1, SW_EC30.1, SW_EC33.1, SW_EC36.1, SW_EC39.1, SW_EC6.1, SW_EC9.1
- net C5: now reaches SW_EC16.2, SW_EC17.2, SW_EC18.2, SW_EC21.2
- net C8: now reaches SW_EC28.2, SW_EC29.2, SW_EC30.2, SW_EC42.2
- net C10: now reaches SW_EC34.2, SW_EC35.2, SW_EC36.2
- net C4: now reaches SW_EC13.2, SW_EC14.2, SW_EC15.2, SW_EC20.2
- net C3: now reaches SW_EC10.2, SW_EC11.2, SW_EC12.2, SW_EC19.2
- net C9: now reaches SW_EC31.2, SW_EC32.2, SW_EC33.2
- net C2: now reaches SW_EC7.2, SW_EC8.2, SW_EC9.2
- net C6: now reaches SW_EC22.2, SW_EC23.2, SW_EC24.2, SW_EC40.2

Commit message: re did the pcb
Parts:
- added SW_EC1, SW_EC13, SW_EC18, SW_EC23, SW_EC28, SW_EC33, SW_EC38, SW_EC43, SW_EC47, SW_EC5, SW_EC51, SW_EC9: Topre, footprints:Topre, symbol cipulot_parts:Topre
- renumbered SW_EC7 to SW_EC10, SW_EC8 to SW_EC11, SW_EC9 to SW_EC12, SW_EC10 to SW_EC14, SW_EC11 to SW_EC15, SW_EC12 to SW_EC16, SW_EC19 to SW_EC17, SW_EC13 to SW_EC19, SW_EC1 to SW_EC2, SW_EC14 to SW_EC20, SW_EC15 to SW_EC21, SW_EC20 to SW_EC22, SW_EC16 to SW_EC24, SW_EC17 to SW_EC25, SW_EC18 to SW_EC26, SW_EC21 to SW_EC27, SW_EC22 to SW_EC29, SW_EC2 to SW_EC3, SW_EC23 to SW_EC30, SW_EC24 to SW_EC31, SW_EC40 to SW_EC32, SW_EC25 to SW_EC34, SW_EC26 to SW_EC35, SW_EC27 to SW_EC36, SW_EC41 to SW_EC37, SW_EC28 to SW_EC39, SW_EC3 to SW_EC4, SW_EC29 to SW_EC40, SW_EC30 to SW_EC41, SW_EC31 to SW_EC44, SW_EC32 to SW_EC45, SW_EC33 to SW_EC46, SW_EC34 to SW_EC48, SW_EC35 to SW_EC49, SW_EC36 to SW_EC50, SW_EC37 to SW_EC52, SW_EC38 to SW_EC53, SW_EC39 to SW_EC54, SW_EC4 to SW_EC6, SW_EC5 to SW_EC7, SW_EC6 to SW_EC8
Connections:
- net C0: now also SW_EC1.2
- net C1: now also SW_EC5.2
- net C10: now also SW_EC47.2
- net C11: now also SW_EC51.2
- net C2: now also SW_EC9.2
- net C3: now also SW_EC13.2
- net C4: now also SW_EC18.2
- net C5: now also SW_EC23.2
- net C6: now also SW_EC28.2
- net C7: now also SW_EC33.2
- net C8: now also SW_EC38.2
- net C9: now also SW_EC43.2
- net GND: now also SW_EC1.3, SW_EC13.3, SW_EC18.3, SW_EC23.3, SW_EC28.3, SW_EC33.3, SW_EC38.3, SW_EC43.3, SW_EC47.3, SW_EC5.3, SW_EC51.3, SW_EC9.3
- net R0: now also SW_EC1.1, SW_EC13.1, SW_EC18.1, SW_EC23.1, SW_EC28.1, SW_EC33.1, SW_EC38.1, SW_EC43.1, SW_EC47.1, SW_EC5.1, SW_EC51.1, SW_EC9.1; no longer SW_EC10.1, SW_EC14.1, SW_EC19.1, SW_EC2.1, SW_EC24.1, SW_EC29.1, SW_EC34.1, SW_EC39.1, SW_EC44.1, SW_EC48.1, SW_EC52.1, SW_EC6.1
- net R1: now also SW_EC10.1, SW_EC14.1, SW_EC19.1, SW_EC2.1, SW_EC24.1, SW_EC29.1, SW_EC34.1, SW_EC39.1, SW_EC44.1, SW_EC48.1, SW_EC52.1, SW_EC6.1; no longer SW_EC11.1, SW_EC15.1, SW_EC20.1, SW_EC25.1, SW_EC3.1, SW_EC30.1, SW_EC35.1, SW_EC40.1, SW_EC45.1, SW_EC49.1, SW_EC53.1, SW_EC7.1
- net R2: now also SW_EC11.1, SW_EC15.1, SW_EC20.1, SW_EC25.1, SW_EC3.1, SW_EC30.1, SW_EC35.1, SW_EC40.1, SW_EC45.1, SW_EC49.1, SW_EC53.1, SW_EC7.1; no longer SW_EC12.1, SW_EC16.1, SW_EC21.1, SW_EC26.1, SW_EC31.1, SW_EC36.1, SW_EC4.1, SW_EC41.1, SW_EC46.1, SW_EC50.1, SW_EC54.1, SW_EC8.1
- net R3: now also SW_EC12.1, SW_EC16.1, SW_EC21.1, SW_EC26.1, SW_EC31.1, SW_EC36.1, SW_EC4.1, SW_EC41.1, SW_EC46.1, SW_EC50.1, SW_EC54.1, SW_EC8.1; no longer SW_EC17.1, SW_EC22.1, SW_EC27.1, SW_EC32.1, SW_EC37.1, SW_EC42.1
- new net R4: SW_EC17.1, SW_EC22.1, SW_EC27.1, SW_EC32.1, SW_EC37.1, SW_EC42.1
